File: EDC_FINAL_PROJECT.kicad_pcb (KiCad board)
At the start: 2 copper layers, 88.9 x 50.8 mm, 31 parts, among them J1 Screw_Terminal_01x02, J2 Screw_Terminal_01x03, SW1 SW_Push_DPDT, U1 LM317_TO-220, U2 LM337_TO220

Commit message: 10.12.2025 rebase
Parts:
- moved U2 61.0 mm to (157.5, 83.3), turned to 0 degrees
- moved C2 45.1 mm to (118.1, 82.4)
- moved C3 44.5 mm to (110.5, 82.4)
- moved J2 40.6 mm to (111.4, 123.2), turned to 0 degrees
- moved C6 20.5 mm to (118.1, 96.3)
- moved D2 8.45 mm to (108.0, 89.4)
- moved D4 8.45 mm to (108.0, 103.3)
- moved D1 8.43 mm to (113.0, 89.4)
- moved D3 8.43 mm to (113.0, 103.3)
- moved RV1 1.39 mm to (144.2, 123.2)
- moved RV2 1.28 mm to (127.7, 123.2)
- moved J1 0.83 mm to (160.7, 123.2)
- moved C5 0.79 mm to (134.0, 115.4)
- moved D10 0.79 mm to (156.2, 104.6)
- moved D6 0.79 mm to (154.3, 90.0)
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
Commit message: rebase_v2 --1
Parts:
- moved U2 56.7 mm to (109.2, 113.0), turned to 90 degrees
- moved C2 43.8 mm to (161.9, 81.9)
- moved C3 43.8 mm to (154.3, 82.0)
- moved D3 11.9 mm to (113.0, 91.4)
- moved D4 11.9 mm to (108.0, 91.4)
- moved D1 9.02 mm to (108.0, 81.9), turned to 0 degrees
- moved C5 2.59 mm to (135.9, 113.6)
- moved D2 2.37 mm to (108.0, 87.0), turned to 0 degrees

Commit message: 10.12.2025 --3
Parts:
- moved C3 2.75 mm to (155.6, 84.4), turned to 90 degrees
Routing:
- net Net-(D10-K): track 0.00 -> 207.4 mm
- net Net-(D10-A): track 0.00 -> 144.7 mm, vias 0 -> 2
- net Net-(D9-K): track 0.00 -> 91.9 mm
- net Net-(D1-A): track 0.00 -> 90.3 mm, vias 0 -> 2
- net Net-(D5-A): track 0.00 -> 77.8 mm
- net Net-(RV1-Pad3): track 0.00 -> 65.6 mm
- net Net-(D6-A): track 0.00 -> 61.9 mm
- net Net-(D1-K): track 0.00 -> 51.7 mm
- net Net-(D2-K): track 0.00 -> 50.8 mm
- net Net-(D11-A): track 0.00 -> 46.9 mm
- net Net-(D3-K): track 0.00 -> 36.3 mm
- net Net-(D12-K): track 0.00 -> 31.4 mm
- net Net-(D12-A): track 0.00 -> 27.5 mm
- net Net-(J1-Pin_2): track 0.00 -> 18.9 mm
- net Net-(RV1-Pad1): track 0.00 -> 11.5 mm
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
Commit message: 10.12.2025 --5
Parts:
- moved U2 57.1 mm to (158.1, 83.5), turned to 0 degrees
- moved C2 45.1 mm to (116.8, 82.6)
- moved C3 45.1 mm to (110.5, 85.0)
- moved D3 13.3 mm to (113.0, 104.8)
- moved D4 13.3 mm to (108.0, 104.8)
- moved D1 9.69 mm to (113.0, 90.2), turned to -90 degrees
- moved D2 3.17 mm to (108.0, 90.2), turned to -90 degrees
- moved U1 0.17 mm to (141.6, 83.5)
Routing:
- net Net-(D5-A): track 77.8 -> 119.4 mm
- net Net-(D2-K): track 50.8 -> 86.0 mm, vias 0 -> 1
- net Net-(D6-A): track 61.9 -> 90.2 mm
- net Net-(D3-K): track 36.3 -> 21.9 mm
- net Net-(D9-K): track 91.9 -> 79.3 mm
- net Net-(D1-K): track 51.7 -> 43.3 mm
- net Net-(RV1-Pad3): track 65.6 -> 72.6 mm, vias 0 -> 1
- net Net-(D1-A): track 90.3 -> 97.1 mm, vias 2 -> 1
- net Net-(D10-A): track 144.7 -> 151.4 mm, vias 2 -> 1
- net Net-(D11-A): track 46.9 -> 44.1 mm
- net Net-(D10-K): track 207.4 -> 208.1 mm

Commit message: 10.12.2025 --7
Parts:
- D10, D5, D6, D7, D8, D9: footprint Diode_THT:D_DO-41_SOD81_P10.16mm_Horizontal -> Diode_THT:D_DO-41_SOD81_P5.08mm_Vertical_AnodeUp
- R1, R2, R3, R4, R5, R6: footprint Resistor_THT:R_Axial_DIN0414_L11.9mm_D4.5mm_P15.24mm_Horizontal -> Resistor_THT:R_Axial_DIN0414_L11.9mm_D4.5mm_P7.62mm_Vertical
- RV2: footprint TerminalBlock_Phoenix:TerminalBlock_Phoenix_MKDS-1,5-3_1x03_P5.00mm_Horizontal -> Potentiometer_THT:Potentiometer_Bourns_3296W_Vertical
- moved R2 67.2 mm to (103.6, 81.0)
- moved D12 62.9 mm to (121.1, 116.1)
- moved U2 62.5 mm to (104.6, 115.8), turned to 180 degrees
- moved R4 61.3 mm to (109.7, 104.9), turned to 0 degrees
- moved D11 53.4 mm to (137.8, 82.3), turned to 180 degrees
- moved U1 53.2 mm to (88.6, 78.5)
- moved R6 49.0 mm to (131.1, 100.7), turned to 0 degrees
- moved J2 47.9 mm to (74.5, 92.5), turned to -90 degrees
- moved D1 47.0 mm to (70.9, 110.9), turned to 0 degrees
- moved R5 46.8 mm to (131.1, 93.7), turned to 0 degrees
- moved D6 46.2 mm to (109.2, 80.3)
- moved RV2 43.5 mm to (125.2, 79.8), turned to 90 degrees
- moved D4 42.7 mm to (70.2, 84.8), turned to 0 degrees
- moved D10 41.7 mm to (115.0, 97.8)
- moved D7 41.4 mm to (118.4, 80.2), turned to -90 degrees
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Routing:
- net Net-(R5-Pad1): track 11.3 -> 101.2 mm
- net Net-(D5-A): track 119.4 -> 189.1 mm
- net Net-(RV1-Pad1): track 11.5 -> 80.9 mm
- net Net-(D10-A): track 151.4 -> 104.5 mm, vias 1 -> 0
- net Net-(D6-A): track 90.2 -> 45.5 mm
- net Net-(D9-K): track 79.3 -> 37.6 mm
- net Net-(D1-K): track 43.3 -> 14.9 mm
- net Net-(D10-K): track 208.1 -> 181.5 mm
- net Net-(J1-Pin_2): track 18.9 -> 41.7 mm
- net Net-(D11-A): track 44.1 -> 24.6 mm
- net Net-(D1-A): track 97.1 -> 78.7 mm, vias 1 -> 0
- net Net-(D12-K): track 31.4 -> 39.6 mm
- net Net-(D3-K): track 21.9 -> 15.2 mm
- net Net-(RV1-Pad3): track 72.6 -> 66.4 mm, vias 1 -> 0
- net Net-(D2-K): track 86.0 -> 89.3 mm, vias 1 -> 0
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
Commit message: 10.12.2025 --final revision
Parts:
- moved D9 11.2 mm to (132.1, 105.2)
- moved U2 10.7 mm to (94.0, 117.1)
- moved R4 10.4 mm to (120.2, 105.2)
- moved D8 9.41 mm to (114.3, 103.4)
- moved C2 3.62 mm to (125.0, 89.2), turned to -90 degrees
- moved D7 2.82 mm to (118.9, 77.5)
- moved D6 2.79 mm to (109.2, 77.5)
- moved R2 2.54 mm to (103.6, 78.5)
- moved D12 2.38 mm to (118.7, 115.8)
- moved R5 1.80 mm to (131.3, 91.9)
- moved R6 1.67 mm to (131.3, 99.1)
- moved C6 1.59 mm to (125.0, 98.5), turned to 90 degrees
- moved D11 1.37 mm to (137.3, 81.0)
- moved R3 1.31 mm to (102.9, 97.3)
- moved RV1 1.14 mm to (148.1, 87.1)
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Routing:
- net Net-(RV1-Pad1): track 80.9 -> 31.0 mm
- net Net-(D10-A): track 104.5 -> 149.9 mm
- net Net-(D5-A): track 189.1 -> 165.0 mm
- net Net-(RV1-Pad3): track 66.4 -> 47.8 mm
- net Net-(D9-K): track 37.6 -> 55.2 mm
- net Net-(R5-Pad1): track 101.2 -> 84.3 mm
- net Net-(D11-A): track 24.6 -> 13.7 mm
- net Net-(D2-K): track 89.3 -> 100.0 mm
- net Net-(D6-A): track 45.5 -> 51.8 mm
- net Net-(D10-K): track 181.5 -> 177.8 mm
- net Net-(D1-A): track 78.7 -> 81.1 mm
- net Net-(J1-Pin_2): track 41.7 -> 40.6 mm
- net Net-(D12-A): track 28.0 -> 29.0 mm
- net Net-(D12-K): track 39.6 -> 38.8 mm
Other:
- board text added: "ROVIC MAGDAMIT BS ECE ECE-201L POWER SUPPLY"

Commit message: 10.14.2025
Parts:
- R1, R3: value 5K1 -> 5K; footprint Resistor_THT:R_Axial_DIN0414_L11.9mm_D4.5mm_P7.62mm_Vertical -> Resistor_THT:R_Axial_DIN0411_L9.9mm_D3.6mm_P7.62mm_Vertical
- R2, R4, R5, R6: footprint Resistor_THT:R_Axial_DIN0414_L11.9mm_D4.5mm_P7.62mm_Vertical -> Resistor_THT:R_Axial_DIN0411_L9.9mm_D3.6mm_P7.62mm_Vertical
- moved D5 32.9 mm to (135.6, 92.6)
- moved J1 32.9 mm to (164.5, 116.7)
- moved RV1 32.9 mm to (181.0, 88.1)
- moved SW1 32.9 mm to (181.0, 119.4)
- moved C2 32.9 mm to (157.9, 90.1)
- moved C5 32.9 mm to (142.6, 97.3)
- moved C6 32.9 mm to (157.9, 99.5)
- moved D1 32.9 mm to (104.3, 111.7)
- moved D12 32.9 mm to (151.6, 116.8)
- moved D2 32.9 mm to (114.4, 116.8)
- moved D3 32.9 mm to (113.8, 80.6)
- moved D4 32.9 mm to (103.6, 85.7)
- moved D6 32.9 mm to (142.1, 78.4)
- moved D7 32.9 mm to (151.8, 78.4)
- moved D8 32.9 mm to (147.2, 104.3)
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Routing:
- net Net-(D10-K): track 177.8 -> 176.9 mm

Commit message: 10.17.2025
Parts:
- D10, D5, D6, D7, D8, D9: footprint Diode_THT:D_DO-41_SOD81_P5.08mm_Vertical_AnodeUp -> Diode_THT:D_DO-41_SOD81_P10.16mm_Horizontal
- R1, R2, R3, R4, R5, R6: footprint Resistor_THT:R_Axial_DIN0411_L9.9mm_D3.6mm_P7.62mm_Vertical -> Resistor_THT:R_Axial_DIN0411_L9.9mm_D3.6mm_P15.24mm_Horizontal
- moved D2 41.1 mm to (103.6, 77.2), turned to -90 degrees
- moved D12 40.3 mm to (185.7, 95.2), turned to 90 degrees
- moved J1 39.7 mm to (185.9, 83.2), turned to 90 degrees
- moved D9 36.0 mm to (129.1, 109.5)
- moved D4 33.7 mm to (104.1, 119.3), turned to 90 degrees
- moved D3 32.8 mm to (97.7, 109.2), turned to -90 degrees
- moved D11 29.6 mm to (185.7, 107.2), turned to 90 degrees
- moved D8 29.0 mm to (122.2, 119.0)
- moved D5 28.3 mm to (111.8, 77.5)
- moved D1 25.3 mm to (97.4, 87.3), turned to 90 degrees
- moved C5 19.0 mm to (160.4, 104.0), turned to 0 degrees
- moved RV2 18.9 mm to (176.6, 83.8), turned to -90 degrees
- moved SW1 18.5 mm to (162.7, 116.8), turned to 0 degrees
- moved C3 18.1 mm to (160.1, 93.0), turned to 0 degrees
- moved R5 16.4 mm to (173.9, 106.1), turned to 90 degrees
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Routing:
- net Net-(D10-K): track 176.9 -> 341.8 mm
- net Net-(R5-Pad1): track 84.3 -> 11.1 mm
- net Net-(D5-A): track 165.0 -> 95.5 mm
- net Net-(D10-A): track 149.9 -> 118.8 mm
- net Net-(D3-K): track 15.3 -> 42.3 mm
- net Net-(RV1-Pad3): track 47.8 -> 71.7 mm
- net Net-(RV1-Pad1): track 31.0 -> 8.79 mm
- net Net-(D1-K): track 14.8 -> 35.4 mm
- net Net-(D2-K): track 100.0 -> 82.8 mm
- net Net-(J1-Pin_2): track 40.6 -> 25.4 mm
- net Net-(D12-K): track 38.8 -> 24.8 mm
- net Net-(D1-A): track 81.1 -> 93.5 mm
- net Net-(D6-A): track 51.8 -> 40.1 mm
- net Net-(D11-A): track 13.7 -> 24.6 mm
- net Net-(D12-A): track 29.0 -> 18.6 mm
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Other:
- board size 88.9 x 50.8 mm -> 101.6 x 50.8 mm
- board text removed: "ROVIC MAGDAMIT BS ECE ECE-201L POWER SUPPLY"
