File: EDC_FINAL_PROJECT.kicad_pcb (KiCad board)
At the start: 2 copper layers, 101.6 x 50.8 mm, 31 parts, among them J1 Screw_Terminal_01x02, J2 Screw_Terminal_01x03, SW1 SW_Push_DPDT, U1 LM317_TO-220, U2 LM337_TO220

Commit message: 10.21.2025
Parts:
- added C1: 2200 uF, Capacitor_THT:CP_Radial_D16.0mm_P7.50mm, F.Cu at (67.2, 150.8)
- added C1: 2200 uF, Capacitor_THT:CP_Radial_D16.0mm_P7.50mm, F.Cu at (67.0, 90.7)
- added C1: 2200 uF, Capacitor_THT:CP_Radial_D16.0mm_P7.50mm, F.Cu at (178.2, 150.3)
- added C1: 2200 uF, Capacitor_THT:CP_Radial_D16.0mm_P7.50mm, F.Cu at (177.9, 90.7)
- added C1: 2200 uF, Capacitor_THT:CP_Radial_D16.0mm_P7.50mm, F.Cu at (177.1, 31.3)
- added C2: 0.1 uF, Capacitor_THT:C_Disc_D5.0mm_W2.5mm_P2.50mm, F.Cu at (215.6, 31.1)
- added C2: 0.1 uF, Capacitor_THT:C_Disc_D5.0mm_W2.5mm_P2.50mm, F.Cu at (216.7, 150.1)
- added C2: 0.1 uF, Capacitor_THT:C_Disc_D5.0mm_W2.5mm_P2.50mm, F.Cu at (105.7, 150.6)
- added C2: 0.1 uF, Capacitor_THT:C_Disc_D5.0mm_W2.5mm_P2.50mm, F.Cu at (105.5, 90.5)
- added C2: 0.1 uF, Capacitor_THT:C_Disc_D5.0mm_W2.5mm_P2.50mm, F.Cu at (216.4, 90.5)
- added C3: 10 uF, Capacitor_THT:CP_Radial_D5.0mm_P2.50mm, F.Cu at (221.7, 158.1)
- added C3: 10 uF, Capacitor_THT:CP_Radial_D5.0mm_P2.50mm, F.Cu at (220.6, 39.1)
- added C3: 10 uF, Capacitor_THT:CP_Radial_D5.0mm_P2.50mm, F.Cu at (110.5, 98.5)
- added C3: 10 uF, Capacitor_THT:CP_Radial_D5.0mm_P2.50mm, F.Cu at (221.4, 98.5)
- added C3: 10 uF, Capacitor_THT:CP_Radial_D5.0mm_P2.50mm, F.Cu at (110.7, 158.6)
- added C4: 2200 uF, Capacitor_THT:CP_Radial_D16.0mm_P7.50mm, F.Cu at (67.2, 169.3)
- added C4: 2200 uF, Capacitor_THT:CP_Radial_D16.0mm_P7.50mm, F.Cu at (177.9, 109.2)
- added C4: 2200 uF, Capacitor_THT:CP_Radial_D16.0mm_P7.50mm, F.Cu at (178.2, 168.8)
- added C4: 2200 uF, Capacitor_THT:CP_Radial_D16.0mm_P7.50mm, F.Cu at (67.0, 109.2)
- added C4: 2200 uF, Capacitor_THT:CP_Radial_D16.0mm_P7.50mm, F.Cu at (177.1, 49.9)
- added C5: 10 uF, Capacitor_THT:CP_Radial_D5.0mm_P2.50mm, F.Cu at (221.7, 109.5)
- added C5: 10 uF, Capacitor_THT:CP_Radial_D5.0mm_P2.50mm, F.Cu at (110.8, 109.5)
- added C5: 10 uF, Capacitor_THT:CP_Radial_D5.0mm_P2.50mm, F.Cu at (110.9, 169.6)
- added C5: 10 uF, Capacitor_THT:CP_Radial_D5.0mm_P2.50mm, F.Cu at (220.9, 50.1)
- added C5: 10 uF, Capacitor_THT:CP_Radial_D5.0mm_P2.50mm, F.Cu at (221.9, 169.1)
- added C6: 0.1 uF, Capacitor_THT:C_Disc_D5.0mm_W2.5mm_P2.50mm, F.Cu at (105.9, 174.8)
- added C6: 0.1 uF, Capacitor_THT:C_Disc_D5.0mm_W2.5mm_P2.50mm, F.Cu at (216.9, 174.3)
- added C6: 0.1 uF, Capacitor_THT:C_Disc_D5.0mm_W2.5mm_P2.50mm, F.Cu at (105.7, 114.8)
- added C6: 0.1 uF, Capacitor_THT:C_Disc_D5.0mm_W2.5mm_P2.50mm, F.Cu at (215.9, 55.4)
- added C6: 0.1 uF, Capacitor_THT:C_Disc_D5.0mm_W2.5mm_P2.50mm, F.Cu at (216.6, 114.8)
- added D1: 1N4007, Diode_THT:D_DO-41_SOD81_P10.16mm_Horizontal, F.Cu at (158.9, 152.4)
- added D1: 1N4007, Diode_THT:D_DO-41_SOD81_P10.16mm_Horizontal, F.Cu at (157.9, 33.4)
- added D1: 1N4007, Diode_THT:D_DO-41_SOD81_P10.16mm_Horizontal, F.Cu at (158.6, 92.8)
- added D1: 1N4007, Diode_THT:D_DO-41_SOD81_P10.16mm_Horizontal, F.Cu at (47.7, 92.8)
- added D1: 1N4007, Diode_THT:D_DO-41_SOD81_P10.16mm_Horizontal, F.Cu at (47.9, 152.9)
- added D10: 1N4007, Diode_THT:D_DO-41_SOD81_P10.16mm_Horizontal, F.Cu at (211.9, 51.3)
- added D10: 1N4007, Diode_THT:D_DO-41_SOD81_P10.16mm_Horizontal, F.Cu at (101.7, 110.7)
- added D10: 1N4007, Diode_THT:D_DO-41_SOD81_P10.16mm_Horizontal, F.Cu at (212.6, 110.7)
- added D10: 1N4007, Diode_THT:D_DO-41_SOD81_P10.16mm_Horizontal, F.Cu at (212.9, 170.2)
- added D10: 1N4007, Diode_THT:D_DO-41_SOD81_P10.16mm_Horizontal, F.Cu at (101.9, 170.7)
- added D11: LED, TerminalBlock_Phoenix:TerminalBlock_Phoenix_MKDS-1,5-2_1x02_P5.00mm_Horizontal, F.Cu at (136.2, 172.8)
- added D11: LED, TerminalBlock_Phoenix:TerminalBlock_Phoenix_MKDS-1,5-2_1x02_P5.00mm_Horizontal, F.Cu at (246.2, 53.4)
- added D11: LED, TerminalBlock_Phoenix:TerminalBlock_Phoenix_MKDS-1,5-2_1x02_P5.00mm_Horizontal, F.Cu at (247.0, 112.8)
- added D11: LED, TerminalBlock_Phoenix:TerminalBlock_Phoenix_MKDS-1,5-2_1x02_P5.00mm_Horizontal, F.Cu at (247.2, 172.3)
- added D11: LED, TerminalBlock_Phoenix:TerminalBlock_Phoenix_MKDS-1,5-2_1x02_P5.00mm_Horizontal, F.Cu at (136.1, 112.8)
- added D12: LED, TerminalBlock_Phoenix:TerminalBlock_Phoenix_MKDS-1,5-2_1x02_P5.00mm_Horizontal, F.Cu at (246.2, 41.4)
- added D12: LED, TerminalBlock_Phoenix:TerminalBlock_Phoenix_MKDS-1,5-2_1x02_P5.00mm_Horizontal, F.Cu at (136.1, 100.8)
- added D12: LED, TerminalBlock_Phoenix:TerminalBlock_Phoenix_MKDS-1,5-2_1x02_P5.00mm_Horizontal, F.Cu at (247.0, 100.8)
- added D12: LED, TerminalBlock_Phoenix:TerminalBlock_Phoenix_MKDS-1,5-2_1x02_P5.00mm_Horizontal, F.Cu at (136.2, 160.8)
- added D12: LED, TerminalBlock_Phoenix:TerminalBlock_Phoenix_MKDS-1,5-2_1x02_P5.00mm_Horizontal, F.Cu at (247.2, 160.3)
- added D2: 1N4007, Diode_THT:D_DO-41_SOD81_P10.16mm_Horizontal, F.Cu at (165.2, 142.2)
- added D2: 1N4007, Diode_THT:D_DO-41_SOD81_P10.16mm_Horizontal, F.Cu at (164.1, 23.3)
- added D2: 1N4007, Diode_THT:D_DO-41_SOD81_P10.16mm_Horizontal, F.Cu at (164.9, 82.7)
- added D2: 1N4007, Diode_THT:D_DO-41_SOD81_P10.16mm_Horizontal, F.Cu at (54.2, 142.7)
- added D2: 1N4007, Diode_THT:D_DO-41_SOD81_P10.16mm_Horizontal, F.Cu at (54.0, 82.7)
- added D3: 1N4007, Diode_THT:D_DO-41_SOD81_P10.16mm_Horizontal, F.Cu at (48.3, 174.7)
- added D3: 1N4007, Diode_THT:D_DO-41_SOD81_P10.16mm_Horizontal, F.Cu at (159.0, 114.7)
- added D3: 1N4007, Diode_THT:D_DO-41_SOD81_P10.16mm_Horizontal, F.Cu at (159.3, 174.2)
- added D3: 1N4007, Diode_THT:D_DO-41_SOD81_P10.16mm_Horizontal, F.Cu at (48.1, 114.7)
- added D3: 1N4007, Diode_THT:D_DO-41_SOD81_P10.16mm_Horizontal, F.Cu at (158.2, 55.3)
- added D4: 1N4007, Diode_THT:D_DO-41_SOD81_P10.16mm_Horizontal, F.Cu at (54.7, 184.9)
- added D4: 1N4007, Diode_THT:D_DO-41_SOD81_P10.16mm_Horizontal, F.Cu at (54.5, 124.8)
- added D4: 1N4007, Diode_THT:D_DO-41_SOD81_P10.16mm_Horizontal, F.Cu at (164.6, 65.4)
- added D4: 1N4007, Diode_THT:D_DO-41_SOD81_P10.16mm_Horizontal, F.Cu at (165.7, 184.4)
- added D4: 1N4007, Diode_THT:D_DO-41_SOD81_P10.16mm_Horizontal, F.Cu at (165.4, 124.8)
- added D5: 1N4007, Diode_THT:D_DO-41_SOD81_P10.16mm_Horizontal, F.Cu at (172.3, 23.6)
- added D5: 1N4007, Diode_THT:D_DO-41_SOD81_P10.16mm_Horizontal, F.Cu at (173.1, 83.0)
- added D5: 1N4007, Diode_THT:D_DO-41_SOD81_P10.16mm_Horizontal, F.Cu at (62.3, 143.1)
- added D5: 1N4007, Diode_THT:D_DO-41_SOD81_P10.16mm_Horizontal, F.Cu at (62.1, 83.0)
- added D5: 1N4007, Diode_THT:D_DO-41_SOD81_P10.16mm_Horizontal, F.Cu at (173.3, 142.6)
- added D6: 1N4007, Diode_THT:D_DO-41_SOD81_P10.16mm_Horizontal, F.Cu at (200.2, 92.5)
- added D6: 1N4007, Diode_THT:D_DO-41_SOD81_P10.16mm_Horizontal, F.Cu at (89.5, 152.6)
- added D6: 1N4007, Diode_THT:D_DO-41_SOD81_P10.16mm_Horizontal, F.Cu at (89.3, 92.5)
- added D6: 1N4007, Diode_THT:D_DO-41_SOD81_P10.16mm_Horizontal, F.Cu at (199.4, 33.1)
- added D6: 1N4007, Diode_THT:D_DO-41_SOD81_P10.16mm_Horizontal, F.Cu at (200.5, 152.1)
- added D7: 1N4007, Diode_THT:D_DO-41_SOD81_P10.16mm_Horizontal, F.Cu at (212.6, 86.2)
- added D7: 1N4007, Diode_THT:D_DO-41_SOD81_P10.16mm_Horizontal, F.Cu at (101.7, 86.2)
- added D7: 1N4007, Diode_THT:D_DO-41_SOD81_P10.16mm_Horizontal, F.Cu at (212.9, 145.7)
- added D7: 1N4007, Diode_THT:D_DO-41_SOD81_P10.16mm_Horizontal, F.Cu at (211.9, 26.8)
- added D7: 1N4007, Diode_THT:D_DO-41_SOD81_P10.16mm_Horizontal, F.Cu at (101.9, 146.2)
- added D8: 1N4007, Diode_THT:D_DO-41_SOD81_P10.16mm_Horizontal, F.Cu at (72.7, 184.6)
- added D8: 1N4007, Diode_THT:D_DO-41_SOD81_P10.16mm_Horizontal, F.Cu at (183.7, 184.1)
- added D8: 1N4007, Diode_THT:D_DO-41_SOD81_P10.16mm_Horizontal, F.Cu at (182.7, 65.1)
- added D8: 1N4007, Diode_THT:D_DO-41_SOD81_P10.16mm_Horizontal, F.Cu at (72.6, 124.5)
- added D8: 1N4007, Diode_THT:D_DO-41_SOD81_P10.16mm_Horizontal, F.Cu at (183.5, 124.5)
- added D9: 1N4007, Diode_THT:D_DO-41_SOD81_P10.16mm_Horizontal, F.Cu at (79.5, 115.0)
- added D9: 1N4007, Diode_THT:D_DO-41_SOD81_P10.16mm_Horizontal, F.Cu at (190.4, 115.0)
- added D9: 1N4007, Diode_THT:D_DO-41_SOD81_P10.16mm_Horizontal, F.Cu at (79.7, 175.0)
- added D9: 1N4007, Diode_THT:D_DO-41_SOD81_P10.16mm_Horizontal, F.Cu at (190.7, 174.5)
- added D9: 1N4007, Diode_THT:D_DO-41_SOD81_P10.16mm_Horizontal, F.Cu at (189.6, 55.6)
- added J1: Screw_Terminal_01x02, TerminalBlock_Phoenix:TerminalBlock_Phoenix_MKDS-1,5-2_1x02_P5.00mm_Horizontal, F.Cu at (247.1, 88.8)
- added J1: Screw_Terminal_01x02, TerminalBlock_Phoenix:TerminalBlock_Phoenix_MKDS-1,5-2_1x02_P5.00mm_Horizontal, F.Cu at (136.2, 88.8)
- added J1: Screw_Terminal_01x02, TerminalBlock_Phoenix:TerminalBlock_Phoenix_MKDS-1,5-2_1x02_P5.00mm_Horizontal, F.Cu at (246.4, 29.4)
- added J1: Screw_Terminal_01x02, TerminalBlock_Phoenix:TerminalBlock_Phoenix_MKDS-1,5-2_1x02_P5.00mm_Horizontal, F.Cu at (136.4, 148.8)
- added J1: Screw_Terminal_01x02, TerminalBlock_Phoenix:TerminalBlock_Phoenix_MKDS-1,5-2_1x02_P5.00mm_Horizontal, F.Cu at (247.4, 148.3)
- added J2: Screw_Terminal_01x03, TerminalBlock_Phoenix:TerminalBlock_Phoenix_MKDS-1,5-3_1x03_P5.00mm_Horizontal, F.Cu at (161.4, 158.3)
- added J2: Screw_Terminal_01x03, TerminalBlock_Phoenix:TerminalBlock_Phoenix_MKDS-1,5-3_1x03_P5.00mm_Horizontal, F.Cu at (161.1, 98.8)
- added J2: Screw_Terminal_01x03, TerminalBlock_Phoenix:TerminalBlock_Phoenix_MKDS-1,5-3_1x03_P5.00mm_Horizontal, F.Cu at (50.2, 98.8)
- added J2: Screw_Terminal_01x03, TerminalBlock_Phoenix:TerminalBlock_Phoenix_MKDS-1,5-3_1x03_P5.00mm_Horizontal, F.Cu at (160.3, 39.4)
- added J2: Screw_Terminal_01x03, TerminalBlock_Phoenix:TerminalBlock_Phoenix_MKDS-1,5-3_1x03_P5.00mm_Horizontal, F.Cu at (50.4, 158.8)
- added R1: 5K, Resistor_THT:R_Axial_DIN0411_L9.9mm_D3.6mm_P15.24mm_Horizontal, F.Cu at (202.7, 39.6)
- added R1: 5K, Resistor_THT:R_Axial_DIN0411_L9.9mm_D3.6mm_P15.24mm_Horizontal, F.Cu at (203.8, 158.6)
- added R1: 5K, Resistor_THT:R_Axial_DIN0411_L9.9mm_D3.6mm_P15.24mm_Horizontal, F.Cu at (203.5, 99.0)
- added R1: 5K, Resistor_THT:R_Axial_DIN0411_L9.9mm_D3.6mm_P15.24mm_Horizontal, F.Cu at (92.8, 159.1)
- added R1: 5K, Resistor_THT:R_Axial_DIN0411_L9.9mm_D3.6mm_P15.24mm_Horizontal, F.Cu at (92.6, 99.0)
- added R2: 120R, Resistor_THT:R_Axial_DIN0411_L9.9mm_D3.6mm_P15.24mm_Horizontal, F.Cu at (207.4, 24.7)
- added R2: 120R, Resistor_THT:R_Axial_DIN0411_L9.9mm_D3.6mm_P15.24mm_Horizontal, F.Cu at (208.4, 143.7)
- added R2: 120R, Resistor_THT:R_Axial_DIN0411_L9.9mm_D3.6mm_P15.24mm_Horizontal, F.Cu at (208.1, 84.1)
- added R2: 120R, Resistor_THT:R_Axial_DIN0411_L9.9mm_D3.6mm_P15.24mm_Horizontal, F.Cu at (97.2, 84.1)
- added R2: 120R, Resistor_THT:R_Axial_DIN0411_L9.9mm_D3.6mm_P15.24mm_Horizontal, F.Cu at (97.4, 144.2)
- added R3: 5K, Resistor_THT:R_Axial_DIN0411_L9.9mm_D3.6mm_P15.24mm_Horizontal, F.Cu at (187.5, 49.6)
- added R3: 5K, Resistor_THT:R_Axial_DIN0411_L9.9mm_D3.6mm_P15.24mm_Horizontal, F.Cu at (77.5, 169.1)
- added R3: 5K, Resistor_THT:R_Axial_DIN0411_L9.9mm_D3.6mm_P15.24mm_Horizontal, F.Cu at (188.5, 168.6)
- added R3: 5K, Resistor_THT:R_Axial_DIN0411_L9.9mm_D3.6mm_P15.24mm_Horizontal, F.Cu at (188.3, 109.0)
- added R3: 5K, Resistor_THT:R_Axial_DIN0411_L9.9mm_D3.6mm_P15.24mm_Horizontal, F.Cu at (77.4, 109.0)
- added R4: 120R, Resistor_THT:R_Axial_DIN0411_L9.9mm_D3.6mm_P15.24mm_Horizontal, F.Cu at (207.4, 49.0)
- added R4: 120R, Resistor_THT:R_Axial_DIN0411_L9.9mm_D3.6mm_P15.24mm_Horizontal, F.Cu at (208.1, 108.4)
- added R4: 120R, Resistor_THT:R_Axial_DIN0411_L9.9mm_D3.6mm_P15.24mm_Horizontal, F.Cu at (97.2, 108.4)
- added R4: 120R, Resistor_THT:R_Axial_DIN0411_L9.9mm_D3.6mm_P15.24mm_Horizontal, F.Cu at (208.4, 168.0)
- added R4: 120R, Resistor_THT:R_Axial_DIN0411_L9.9mm_D3.6mm_P15.24mm_Horizontal, F.Cu at (97.4, 168.5)
- added R5: 3K3, Resistor_THT:R_Axial_DIN0411_L9.9mm_D3.6mm_P15.24mm_Horizontal, F.Cu at (235.1, 111.6)
- added R5: 3K3, Resistor_THT:R_Axial_DIN0411_L9.9mm_D3.6mm_P15.24mm_Horizontal, F.Cu at (124.4, 171.7)
- added R5: 3K3, Resistor_THT:R_Axial_DIN0411_L9.9mm_D3.6mm_P15.24mm_Horizontal, F.Cu at (234.4, 52.2)
- added R5: 3K3, Resistor_THT:R_Axial_DIN0411_L9.9mm_D3.6mm_P15.24mm_Horizontal, F.Cu at (124.2, 111.6)
- added R5: 3K3, Resistor_THT:R_Axial_DIN0411_L9.9mm_D3.6mm_P15.24mm_Horizontal, F.Cu at (235.4, 171.2)
- added R6: 3K3, Resistor_THT:R_Axial_DIN0411_L9.9mm_D3.6mm_P15.24mm_Horizontal, F.Cu at (230.2, 171.2)
- added R6: 3K3, Resistor_THT:R_Axial_DIN0411_L9.9mm_D3.6mm_P15.24mm_Horizontal, F.Cu at (119.0, 111.6)
- added R6: 3K3, Resistor_THT:R_Axial_DIN0411_L9.9mm_D3.6mm_P15.24mm_Horizontal, F.Cu at (229.1, 52.2)
- added R6: 3K3, Resistor_THT:R_Axial_DIN0411_L9.9mm_D3.6mm_P15.24mm_Horizontal, F.Cu at (229.9, 111.6)
- added R6: 3K3, Resistor_THT:R_Axial_DIN0411_L9.9mm_D3.6mm_P15.24mm_Horizontal, F.Cu at (119.2, 171.7)
- added RV1: 50K, TerminalBlock_Phoenix:TerminalBlock_Phoenix_MKDS-1,5-3_1x03_P5.00mm_Horizontal, F.Cu at (231.6, 86.2)
- added RV1: 50K, TerminalBlock_Phoenix:TerminalBlock_Phoenix_MKDS-1,5-3_1x03_P5.00mm_Horizontal, F.Cu at (120.7, 86.2)
- added RV1: 50K, TerminalBlock_Phoenix:TerminalBlock_Phoenix_MKDS-1,5-3_1x03_P5.00mm_Horizontal, F.Cu at (230.9, 26.9)
- added RV1: 50K, TerminalBlock_Phoenix:TerminalBlock_Phoenix_MKDS-1,5-3_1x03_P5.00mm_Horizontal, F.Cu at (120.9, 146.3)
- added RV1: 50K, TerminalBlock_Phoenix:TerminalBlock_Phoenix_MKDS-1,5-3_1x03_P5.00mm_Horizontal, F.Cu at (231.9, 145.8)
- added RV2: 2K, Potentiometer_THT:Potentiometer_Bourns_3296W_Vertical, F.Cu at (237.9, 89.2)
- added RV2: 2K, Potentiometer_THT:Potentiometer_Bourns_3296W_Vertical, F.Cu at (127.0, 89.2)
- added RV2: 2K, Potentiometer_THT:Potentiometer_Bourns_3296W_Vertical, F.Cu at (238.2, 148.8)
- added RV2: 2K, Potentiometer_THT:Potentiometer_Bourns_3296W_Vertical, F.Cu at (237.1, 29.9)
- added RV2: 2K, Potentiometer_THT:Potentiometer_Bourns_3296W_Vertical, F.Cu at (127.2, 149.3)
- added SW1: SW_Push_DPDT, TerminalBlock_Phoenix:TerminalBlock_Phoenix_MKDS-1,5-6_1x06_P5.00mm_Horizontal, F.Cu at (224.0, 122.2)
- added SW1: SW_Push_DPDT, TerminalBlock_Phoenix:TerminalBlock_Phoenix_MKDS-1,5-6_1x06_P5.00mm_Horizontal, F.Cu at (113.2, 182.3)
- added SW1: SW_Push_DPDT, TerminalBlock_Phoenix:TerminalBlock_Phoenix_MKDS-1,5-6_1x06_P5.00mm_Horizontal, F.Cu at (224.2, 181.8)
- added SW1: SW_Push_DPDT, TerminalBlock_Phoenix:TerminalBlock_Phoenix_MKDS-1,5-6_1x06_P5.00mm_Horizontal, F.Cu at (113.1, 122.2)
- added SW1: SW_Push_DPDT, TerminalBlock_Phoenix:TerminalBlock_Phoenix_MKDS-1,5-6_1x06_P5.00mm_Horizontal, F.Cu at (223.2, 62.9)
- added U1: LM317_TO-220, Package_TO_SOT_THT:TO-220-3_Vertical, F.Cu at (192.8, 86.5)
- added U1: LM317_TO-220, Package_TO_SOT_THT:TO-220-3_Vertical, F.Cu at (82.1, 146.5)
- added U1: LM317_TO-220, Package_TO_SOT_THT:TO-220-3_Vertical, F.Cu at (192.1, 27.1)
- added U1: LM317_TO-220, Package_TO_SOT_THT:TO-220-3_Vertical, F.Cu at (193.1, 146.0)
- added U1: LM317_TO-220, Package_TO_SOT_THT:TO-220-3_Vertical, F.Cu at (81.9, 86.5)
- added U2: LM337_TO220, Package_TO_SOT_THT:TO-220-3_Vertical, F.Cu at (87.1, 122.0)
- added U2: LM337_TO220, Package_TO_SOT_THT:TO-220-3_Vertical, F.Cu at (198.3, 181.5)
- added U2: LM337_TO220, Package_TO_SOT_THT:TO-220-3_Vertical, F.Cu at (197.2, 62.6)
- added U2: LM337_TO220, Package_TO_SOT_THT:TO-220-3_Vertical, F.Cu at (87.3, 182.0)
- added U2: LM337_TO220, Package_TO_SOT_THT:TO-220-3_Vertical, F.Cu at (198.0, 122.0)
- moved D2 72.5 mm to (54.1, 24.3)
- moved J1 72.5 mm to (136.3, 30.4)
- moved R1 72.5 mm to (92.7, 40.6)
- moved U1 72.5 mm to (82.1, 28.1)
- moved U2 72.5 mm to (87.2, 63.6)
- moved C1 72.5 mm to (67.1, 32.3)
- moved C2 72.5 mm to (105.6, 32.1)
- moved C3 72.5 mm to (110.6, 40.1)
- moved C4 72.5 mm to (67.1, 50.9)
- moved C6 72.5 mm to (105.8, 56.4)
- moved D1 72.5 mm to (47.8, 34.4)
- moved D10 72.5 mm to (101.8, 52.3)
- moved D3 72.5 mm to (48.2, 56.3)
- moved D4 72.5 mm to (54.6, 66.4)
- moved D5 72.5 mm to (62.3, 24.6)
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Connections:
- net Net-(D10-K) renamed GND
Routing:
- net GND: track 341.8 -> 2050.5 mm
- net Net-(D10-A): track 118.8 -> 713.1 mm
- net Net-(D5-A): track 95.5 -> 573.2 mm
- net Net-(D1-A): track 93.5 -> 561.1 mm
- net Net-(D2-K): track 82.8 -> 496.7 mm
- net Net-(RV1-Pad3): track 71.7 -> 430.4 mm
- net Net-(D9-K): track 47.0 -> 281.8 mm
- net Net-(D3-K): track 42.3 -> 253.6 mm
- net Net-(D6-A): track 40.1 -> 240.6 mm
- net Net-(D1-K): track 35.4 -> 212.5 mm
- net Net-(J1-Pin_2): track 25.4 -> 152.5 mm
- net Net-(D12-K): track 24.8 -> 148.9 mm
- net Net-(D11-A): track 24.6 -> 147.9 mm
- net Net-(D12-A): track 18.6 -> 111.8 mm
- net Net-(R5-Pad1): track 11.1 -> 66.7 mm
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- added copper zone on B.Cu, net GND
Other:
- board size 101.6 x 50.8 mm -> 212.8 x 170.3 mm
- board text added: "original"

Commit message: version 1.3.3
Parts:
- removed the C1 at (67.2, 150.8)
- removed the C1 at (67.0, 90.7)
- removed the C1 at (178.2, 150.3)
- removed the C1 at (177.9, 90.7)
- removed the C1 at (177.1, 31.3)
- removed the C2 at (215.6, 31.1)
- removed the C2 at (216.7, 150.1)
- removed the C2 at (105.7, 150.6)
- removed the C2 at (105.5, 90.5)
- removed the C2 at (216.4, 90.5)
- removed the C3 at (221.7, 158.1)
- removed the C3 at (220.6, 39.1)
- removed the C3 at (110.5, 98.5)
- removed the C3 at (221.4, 98.5)
- removed the C3 at (110.7, 158.6)
- removed the C4 at (67.2, 169.3)
- removed the C4 at (177.9, 109.2)
- removed the C4 at (178.2, 168.8)
- removed the C4 at (67.0, 109.2)
- removed the C4 at (177.1, 49.9)
- removed the C5 at (221.7, 109.5)
- removed the C5 at (110.8, 109.5)
- removed the C5 at (110.9, 169.6)
- removed the C5 at (220.9, 50.1)
- removed the C5 at (221.9, 169.1)
- removed the C6 at (105.9, 174.8)
- removed the C6 at (216.9, 174.3)
- removed the C6 at (105.7, 114.8)
- removed the C6 at (215.9, 55.4)
- removed the C6 at (216.6, 114.8)
- removed the D1 at (158.9, 152.4)
- removed the D1 at (157.9, 33.4)
- removed the D1 at (158.6, 92.8)
- removed the D1 at (47.7, 92.8)
- removed the D1 at (47.9, 152.9)
- removed the D10 at (211.9, 51.3)
- removed the D10 at (101.7, 110.7)
- removed the D10 at (212.6, 110.7)
- removed the D10 at (212.9, 170.2)
- removed the D10 at (101.9, 170.7)
- removed the D11 at (136.2, 172.8)
- removed the D11 at (246.2, 53.4)
- removed the D11 at (247.0, 112.8)
- removed the D11 at (247.2, 172.3)
- removed the D11 at (136.1, 112.8)
- removed the D12 at (246.2, 41.4)
- removed the D12 at (136.1, 100.8)
- removed the D12 at (247.0, 100.8)
- removed the D12 at (136.2, 160.8)
- removed the D12 at (247.2, 160.3)
- removed the D2 at (165.2, 142.2)
- removed the D2 at (164.1, 23.3)
- removed the D2 at (164.9, 82.7)
- removed the D2 at (54.2, 142.7)
- removed the D2 at (54.0, 82.7)
- removed the D3 at (48.3, 174.7)
- removed the D3 at (159.0, 114.7)
- removed the D3 at (159.3, 174.2)
- removed the D3 at (48.1, 114.7)
- removed the D3 at (158.2, 55.3)
- removed the D4 at (54.7, 184.9)
- removed the D4 at (54.5, 124.8)
- removed the D4 at (164.6, 65.4)
- removed the D4 at (165.7, 184.4)
- removed the D4 at (165.4, 124.8)
- removed the D5 at (172.3, 23.6)
- removed the D5 at (173.1, 83.0)
- removed the D5 at (62.3, 143.1)
- removed the D5 at (62.1, 83.0)
- removed the D5 at (173.3, 142.6)
- removed the D6 at (200.2, 92.5)
- removed the D6 at (89.5, 152.6)
- removed the D6 at (89.3, 92.5)
- removed the D6 at (199.4, 33.1)
- removed the D6 at (200.5, 152.1)
- removed the D7 at (212.6, 86.2)
- removed the D7 at (101.7, 86.2)
- removed the D7 at (212.9, 145.7)
- removed the D7 at (211.9, 26.8)
- removed the D7 at (101.9, 146.2)
- removed the D8 at (72.7, 184.6)
- removed the D8 at (183.7, 184.1)
- removed the D8 at (182.7, 65.1)
- removed the D8 at (72.6, 124.5)
- removed the D8 at (183.5, 124.5)
- removed the D9 at (79.5, 115.0)
- removed the D9 at (190.4, 115.0)
- removed the D9 at (79.7, 175.0)
- removed the D9 at (190.7, 174.5)
- removed the D9 at (189.6, 55.6)
- removed the J1 at (247.1, 88.8)
- removed the J1 at (136.2, 88.8)
- removed the J1 at (246.4, 29.4)
- removed the J1 at (136.4, 148.8)
- removed the J1 at (247.4, 148.3)
- removed the J2 at (161.4, 158.3)
- removed the J2 at (161.1, 98.8)
- removed the J2 at (50.2, 98.8)
- removed the J2 at (160.3, 39.4)
- removed the J2 at (50.4, 158.8)
- removed the R1 at (202.7, 39.6)
- removed the R1 at (203.8, 158.6)
- removed the R1 at (203.5, 99.0)
- removed the R1 at (92.8, 159.1)
- removed the R1 at (92.6, 99.0)
- removed the R2 at (207.4, 24.7)
- removed the R2 at (208.4, 143.7)
- removed the R2 at (208.1, 84.1)
- removed the R2 at (97.2, 84.1)
- removed the R2 at (97.4, 144.2)
- removed the R3 at (187.5, 49.6)
- removed the R3 at (77.5, 169.1)
- removed the R3 at (188.5, 168.6)
- removed the R3 at (188.3, 109.0)
- removed the R3 at (77.4, 109.0)
- removed the R4 at (207.4, 49.0)
- removed the R4 at (208.1, 108.4)
- removed the R4 at (97.2, 108.4)
- removed the R4 at (208.4, 168.0)
- removed the R4 at (97.4, 168.5)
- removed the R5 at (235.1, 111.6)
- removed the R5 at (124.4, 171.7)
- removed the R5 at (234.4, 52.2)
- removed the R5 at (124.2, 111.6)
- removed the R5 at (235.4, 171.2)
- removed the R6 at (230.2, 171.2)
- removed the R6 at (119.0, 111.6)
- removed the R6 at (229.1, 52.2)
- removed the R6 at (229.9, 111.6)
- removed the R6 at (119.2, 171.7)
- removed the RV1 at (231.6, 86.2)
- removed the RV1 at (120.7, 86.2)
- removed the RV1 at (230.9, 26.9)
- removed the RV1 at (120.9, 146.3)
- removed the RV1 at (231.9, 145.8)
- removed the RV2 at (237.9, 89.2)
- removed the RV2 at (127.0, 89.2)
- removed the RV2 at (238.2, 148.8)
- removed the RV2 at (237.1, 29.9)
- removed the RV2 at (127.2, 149.3)
- removed the SW1 at (224.0, 122.2)
- removed the SW1 at (113.2, 182.3)
- removed the SW1 at (224.2, 181.8)
- removed the SW1 at (113.1, 122.2)
- removed the SW1 at (223.2, 62.9)
- removed the U1 at (192.8, 86.5)
- removed the U1 at (82.1, 146.5)
- removed the U1 at (192.1, 27.1)
- removed the U1 at (193.1, 146.0)
- removed the U1 at (81.9, 86.5)
- removed the U2 at (87.1, 122.0)
- removed the U2 at (198.3, 181.5)
- removed the U2 at (197.2, 62.6)
- removed the U2 at (87.3, 182.0)
- removed the U2 at (198.0, 122.0)
- moved D1 62.4 mm to (86.5, 83.5)
- moved D7 62.4 mm to (140.5, 76.8)
- moved R2 62.4 mm to (136.0, 74.8)
- moved R4 62.4 mm to (136.0, 99.0)
- moved R5 62.4 mm to (163.0, 102.3)
- moved R6 62.4 mm to (157.7, 102.3)
- moved U1 62.4 mm to (120.7, 77.1)
- moved U2 62.4 mm to (125.8, 112.6)
- moved C2 62.4 mm to (144.2, 81.1)
- moved C3 62.4 mm to (149.2, 89.1)
- moved C6 62.4 mm to (144.5, 105.4)
- moved D10 62.4 mm to (140.5, 101.3)
- moved D3 62.4 mm to (86.8, 105.3)
- moved D5 62.4 mm to (100.9, 73.6)
- moved J1 62.4 mm to (175.0, 79.4)
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Routing:
- net GND: track 2050.5 -> 341.8 mm
- net Net-(D10-A): track 713.1 -> 118.8 mm
- net Net-(D5-A): track 573.2 -> 95.5 mm
- net Net-(D1-A): track 561.1 -> 93.5 mm
- net Net-(D2-K): track 496.7 -> 82.8 mm
- net Net-(RV1-Pad3): track 430.4 -> 71.7 mm
- net Net-(D9-K): track 281.8 -> 47.0 mm
- net Net-(D3-K): track 253.6 -> 42.3 mm
- net Net-(D6-A): track 240.6 -> 40.1 mm
- net Net-(D1-K): track 212.5 -> 35.4 mm
- net Net-(J1-Pin_2): track 152.5 -> 25.4 mm
- net Net-(D12-K): track 148.9 -> 24.8 mm
- net Net-(D11-A): track 147.9 -> 24.6 mm
- net Net-(D12-A): track 111.8 -> 18.6 mm
- net Net-(R5-Pad1): track 66.7 -> 11.1 mm
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Other:
- board size 212.8 x 170.3 mm -> 101.6 x 50.8 mm
